File: Hardware/BMS/cell_tps.kicad_sch (KiCad schematic)
At the start: 15 parts

Commit message: begin layout
Parts:
- renumbered TP13 to TP801, TP20 to TP802, TP14 to TP803, TP21 to TP804, TP15 to TP805, TP22 to TP806, TP16 to TP807, TP23 to TP808, TP17 to TP809, TP24 to TP810, TP18 to TP811, TP25 to TP812, TP19 to TP813, TP26 to TP814, TP27 to TP815
Changed lines of the file:
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@@
 		(dnp no)
 		(fields_autoplaced yes)
-		(property "Reference" "TP16"
+		(property "Reference" "TP807"
 			(at 96.52 34.7979 0)
 			(effects
@@
 			(project "bms"
 				(path "/36848c1b-92a5-46b0-877b-0db2387c679c/826e6c70-848d-4f04-803e-a5eb891d5409/e1025dcc-ecdc-4fd2-8475-11da7bf22bb3"
-					(reference "TP16")
+					(reference "TP807")
 					(unit 1)
 				)
@@
 		(dnp no)
 		(fields_autoplaced yes)
-		(property "Reference" "TP13"
+		(property "Reference" "TP801"
 			(at 41.91 34.7979 0)
 			(effects
@@
 			(project "bms"
 				(path "/36848c1b-92a5-46b0-877b-0db2387c679c/826e6c70-848d-4f04-803e-a5eb891d5409/e1025dcc-ecdc-4fd2-8475-11da7bf22bb3"
-					(reference "TP13")
+					(reference "TP801")
 					(unit 1)
 				)
@@
 		(dnp no)
 		(fields_autoplaced yes)
-		(property "Reference" "TP24"
+		(property "Reference" "TP810"
 			(at 114.3 55.1179 0)
 			(effects
@@
 			(project "bms"
 				(path "/36848c1b-92a5-46b0-877b-0db2387c679c/826e6c70-848d-4f04-803e-a5eb891d5409/e1025dcc-ecdc-4fd2-8475-11da7bf22bb3"
-					(reference "TP24")
+					(reference "TP810")
 					(unit 1)
 				)
@@
 		(dnp no)
 		(fields_autoplaced yes)
-		(property "Reference" "TP20"
+		(property "Reference" "TP802"
 			(at 41.91 55.1179 0)
 			(effects
@@
 			(project "bms"
 				(path "/36848c1b-92a5-46b0-877b-0db2387c679c/826e6c70-848d-4f04-803e-a5eb891d5409/e1025dcc-ecdc-4fd2-8475-11da7bf22bb3"
-					(reference "TP20")
+					(reference "TP802")
 					(unit 1)
 				)
@@
 		(dnp no)
 		(fields_autoplaced yes)
-		(property "Reference" "TP14"
+		(property "Reference" "TP803"
 			(at 59.69 34.7979 0)
 			(effects
@@
 			(project "bms"
 				(path "/36848c1b-92a5-46b0-877b-0db2387c679c/826e6c70-848d-4f04-803e-a5eb891d5409/e1025dcc-ecdc-4fd2-8475-11da7bf22bb3"
-					(reference "TP14")
+					(reference "TP803")
 					(unit 1)
 				)
@@
 		(dnp no)
 		(fields_autoplaced yes)
-		(property "Reference" "TP22"
+		(property "Reference" "TP806"
 			(at 78.74 55.1179 0)
 			(effects
@@
 			(project "bms"
 				(path "/36848c1b-92a5-46b0-877b-0db2387c679c/826e6c70-848d-4f04-803e-a5eb891d5409/e1025dcc-ecdc-4fd2-8475-11da7bf22bb3"
-					(reference "TP22")
+					(reference "TP806")
 					(unit 1)
 				)
@@
 		(dnp no)
 		(fields_autoplaced yes)
-		(property "Reference" "TP19"
+		(property "Reference" "TP813"
 			(at 149.86 34.7979 0)
 			(effects
@@
 			(project "bms"
 				(path "/36848c1b-92a5-46b0-877b-0db2387c679c/826e6c70-848d-4f04-803e-a5eb891d5409/e1025dcc-ecdc-4fd2-8475-11da7bf22bb3"
-					(reference "TP19")
+					(reference "TP813")
 					(unit 1)
 				)
@@
 		(dnp no)
 		(fields_autoplaced yes)
-		(property "Reference" "TP21"
+		(property "Reference" "TP804"
 			(at 59.69 55.1179 0)
 			(effects
@@
 			(project "bms"
 				(path "/36848c1b-92a5-46b0-877b-0db2387c679c/826e6c70-848d-4f04-803e-a5eb891d5409/e1025dcc-ecdc-4fd2-8475-11da7bf22bb3"
-					(reference "TP21")
+					(reference "TP804")
 					(unit 1)
 				)
@@
 		(dnp no)
 		(fields_autoplaced yes)
-		(property "Reference" "TP18"
+		(property "Reference" "TP811"
 			(at 132.08 34.7979 0)
 			(effects
@@
 			(project "bms"
 				(path "/36848c1b-92a5-46b0-877b-0db2387c679c/826e6c70-848d-4f04-803e-a5eb891d5409/e1025dcc-ecdc-4fd2-8475-11da7bf22bb3"
-					(reference "TP18")
+					(reference "TP811")
 					(unit 1)
 				)
@@
 		(dnp no)
 		(fields_autoplaced yes)
-		(property "Reference" "TP25"
+		(property "Reference" "TP812"
 			(at 132.08 55.1179 0)
 			(effects
@@
 			(project "bms"
 				(path "/36848c1b-92a5-46b0-877b-0db2387c679c/826e6c70-848d-4f04-803e-a5eb891d5409/e1025dcc-ecdc-4fd2-8475-11da7bf22bb3"
-					(reference "TP25")
+					(reference "TP812")
 					(unit 1)
 				)
@@
 		(dnp no)
 		(fields_autoplaced yes)
-		(property "Reference" "TP17"
+		(property "Reference" "TP809"
 			(at 114.3 34.7979 0)
 			(effects
@@
 			(project "bms"
 				(path "/36848c1b-92a5-46b0-877b-0db2387c679c/826e6c70-848d-4f04-803e-a5eb891d5409/e1025dcc-ecdc-4fd2-8475-11da7bf22bb3"
-					(reference "TP17")
+					(reference "TP809")
 					(unit 1)
 				)
@@
 		(dnp no)
 		(fields_autoplaced yes)
-		(property "Reference" "TP26"
+		(property "Reference" "TP814"
 			(at 149.86 55.1179 0)
 			(effects
@@
 			(project "bms"
 				(path "/36848c1b-92a5-46b0-877b-0db2387c679c/826e6c70-848d-4f04-803e-a5eb891d5409/e1025dcc-ecdc-4fd2-8475-11da7bf22bb3"
-					(reference "TP26")
+					(reference "TP814")
 					(unit 1)
 				)
@@
 		(dnp no)
 		(fields_autoplaced yes)
-		(property "Reference" "TP15"
+		(property "Reference" "TP805"
 			(at 78.74 34.7979 0)
 			(effects
@@
 			(project "bms"
 				(path "/36848c1b-92a5-46b0-877b-0db2387c679c/826e6c70-848d-4f04-803e-a5eb891d5409/e1025dcc-ecdc-4fd2-8475-11da7bf22bb3"
-					(reference "TP15")
+					(reference "TP805")
 					(unit 1)
 				)
@@
 		(dnp no)
 		(fields_autoplaced yes)
-		(property "Reference" "TP23"
+		(property "Reference" "TP808"
 			(at 96.52 55.1179 0)
 			(effects
@@
 			(project "bms"
 				(path "/36848c1b-92a5-46b0-877b-0db2387c679c/826e6c70-848d-4f04-803e-a5eb891d5409/e1025dcc-ecdc-4fd2-8475-11da7bf22bb3"
-					(reference "TP23")
+					(reference "TP808")
 					(unit 1)
 				)
@@
 		(dnp no)
 		(fields_autoplaced yes)
-		(property "Reference" "TP27"
+		(property "Reference" "TP815"
 			(at 173.99 46.2279 0)
 			(effects
@@
 			(project "bms"
 				(path "/36848c1b-92a5-46b0-877b-0db2387c679c/826e6c70-848d-4f04-803e-a5eb891d5409/e1025dcc-ecdc-4fd2-8475-11da7bf22bb3"
-					(reference "TP27")
-					(unit 1)
-				)
+					(reference "TP815")
+					(unit 1)
+				)
