File: Hardware/BMS/filter_balance.kicad_sch (KiCad schematic)
At the start: 5 parts

Commit message: edits to the BMS
Parts:
- added D201: WHITE, LED_SMD:LED_0805_2012Metric, symbol Device:LED
- added R202: 100, Resistor_SMD:R_0603_1608Metric, symbol Device:R
- R201: renamed from R8; value 26 -> 33
- renumbered C3 to C201, F3 to F201, JP3 to JP201, R9 to R203
Connections:
- net SN: now also R202.1
- net at F201.2, R201.1, R203.1: now also D201.2 (A)
- new net: D201.1 (K), R202.2
