File: Hardware/BMS/leds.kicad_sch (KiCad schematic)
At the start: 24 parts

Commit message: begin layout
Parts:
- renumbered D1 to D1101, D11 to D1102, D17 to D1103, D5 to D1104, D12 to D1105, D6 to D1106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
