File: Hardware/BMS/power.kicad_sch (KiCad schematic)
At the start: 33 parts, among them Q501 SQ2337ES

Commit message: begin layout
Parts:
- renumbered C501 to C601, C502 to C602, C503 to C603, C504 to C604, C505 to C605, C506 to C606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
