File: Hardware/BMS/therm_tps.kicad_sch (KiCad schematic)
At the start: 28 parts

Commit message: begin layout
Parts:
- renumbered TP28 to TP901, TP32 to TP902, TP36 to TP903, TP40 to TP904, TP44 to TP905, TP48 to TP906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
