File: Hardware/BMS/bms.kicad_pcb (KiCad board)
At the start: 2 copper layers, 78 parts, among them J1 Conn_02x09_Counter_Clockwise, U1 ADBMS1818, U3 MAX33011EASA, U5 STM32G473CCTx

Commit message: begin layout
Parts:
- removed C1, C10, C11, C12, C13, C14, C2, C3, C4, C5, C6, C7, C8, C9: C_10nF, OEM:C_0603_1608Metric
- removed C15: C_0.1uF, OEM:C_0603_1608Metric
- removed F1, F10, F11, F12, F13, F14, F2, F3, F4, F5, F6, F7, F8, F9: 200mA_Fuse, Fuse:Fuse_1206_3216Metric
- removed J1: Conn_02x09_Counter_Clockwise, Connector_PinSocket_2.54mm:PinSocket_2x09_P2.54mm_Vertical
- removed JP1, JP10, JP11, JP12, JP13, JP14, JP2, JP3, JP4, JP5, JP6, JP7, JP8, JP9: SolderJumper_2_Open, Jumper:SolderJumper-2_P1.3mm_Open_TrianglePad1.0x1.5mm
- removed R11, R14, R17, R2, R20, R23, R26, R37, R40, R43, R46, R49, R5, R8: 26, Resistor_SMD:R_2512_6332Metric
- removed R12, R15, R18, R21, R24, R27, R3, R30, R38, R41, R44, R47, R50, R6, R9: 100, OEM:R_0603_1608Metric
- removed R29: 20k, OEM:R_0603_1608Metric
- removed R31: R_120_DNP, OEM:R_0603_1608Metric
- removed U1: ADBMS1818, OEM:LQFP-64-1EP_12x12_P0.5
- removed U3: MAX33011EASA, OEM:SOIC-8_3.9x4.9mm_Pitch1.27mm_OEM
- removed U5: STM32G473CCTx, Package_QFP:LQFP-48_7x7mm_P0.5mm
- added C1001: C_10nF, OEM:C_0603_1608Metric, F.Cu at (42.0, 98.0)
- added C101: C_0.1uF, OEM:C_0603_1608Metric, F.Cu at (45.1, 46.5)
- added C102: C_0.1uF, OEM:C_0603_1608Metric, F.Cu at (45.1, 49.0)
- added C1201: C_10nF, OEM:C_0603_1608Metric, F.Cu at (27.1, 83.6)
- added C1301: C_10nF, OEM:C_0603_1608Metric, F.Cu at (84.6, 120.3)
- added C1401: C_10nF, OEM:C_0603_1608Metric, F.Cu at (42.0, 69.1)
- added C1501: C_10nF, OEM:C_0603_1608Metric, F.Cu at (27.1, 69.1)
- added C1601: C_10nF, OEM:C_0603_1608Metric, F.Cu at (27.1, 98.0)
- added C1701: C_10nF, OEM:C_0603_1608Metric, F.Cu at (115.8, 28.7)
- added C1801: C_10nF, OEM:C_0603_1608Metric, F.Cu at (115.6, 97.2)
- added C1901: C_10nF, OEM:C_0603_1608Metric, F.Cu at (101.0, 43.2)
- added C2001: C_10nF, OEM:C_0603_1608Metric, F.Cu at (42.0, 83.6)
- added C201: C_10nF, OEM:C_0603_1608Metric, F.Cu at (27.1, 112.5)
- added C2101: C_10nF, OEM:C_0603_1608Metric, F.Cu at (115.6, 111.7)
- added C2201: C_10nF, OEM:C_0603_1608Metric, F.Cu at (115.8, 43.2)
- added C301: 1uF, Capacitor_SMD:C_0603_1608Metric, F.Cu at (74.9, 23.8)
- added C302: 1uF, Capacitor_SMD:C_0603_1608Metric, F.Cu at (74.9, 26.3)
- added C303: 1uF, Capacitor_SMD:C_0603_1608Metric, F.Cu at (74.9, 28.8)
- added C304: 1uF, Capacitor_SMD:C_0603_1608Metric, F.Cu at (74.9, 31.3)
- added C305: 0.1uF, Capacitor_SMD:C_0603_1608Metric, F.Cu at (74.9, 33.9)
- added C306: 0.1uF, Capacitor_SMD:C_0603_1608Metric, F.Cu at (74.9, 36.4)
- added C307: 1uF, Capacitor_SMD:C_0603_1608Metric, F.Cu at (74.9, 38.9)
- added C308: 1uF, Capacitor_SMD:C_0603_1608Metric, F.Cu at (78.9, 23.8)
- added C401: C_8pF, OEM:C_0603_1608Metric, F.Cu at (95.1, 56.5)
- added C402: C_8pF, OEM:C_0603_1608Metric, F.Cu at (95.1, 59.0)
- added C403: C_0.1uF, OEM:C_0603_1608Metric, F.Cu at (95.1, 61.5)
- added C404: C_0.1uF, OEM:C_0603_1608Metric, F.Cu at (95.1, 64.0)
- added C405: C_0.1uF, OEM:C_0603_1608Metric, F.Cu at (95.1, 66.5)
- added C406: 100nF, Capacitor_SMD:C_0603_1608Metric, F.Cu at (95.1, 69.0)
- added C407: C_100nF, OEM:C_0603_1608Metric, F.Cu at (95.1, 71.5)
- added C408: 100nF, Capacitor_SMD:C_0603_1608Metric, F.Cu at (99.1, 56.5)
- added C409: 100nF, Capacitor_SMD:C_0603_1608Metric, F.Cu at (99.1, 59.0)
- added C410: 1uF, Capacitor_SMD:C_0603_1608Metric, F.Cu at (99.1, 61.5)
- added C411: 100nF, Capacitor_SMD:C_0603_1608Metric, F.Cu at (99.1, 64.0)
- added C412: C_100nF, OEM:C_0603_1608Metric, F.Cu at (99.1, 66.5)
- added C413: 4.7uF, Capacitor_SMD:C_0805_2012Metric, F.Cu at (123.6, 56.7)
- added C414: 1uF, Capacitor_SMD:C_0603_1608Metric, F.Cu at (99.1, 69.0)
- added C415: 10uF, Capacitor_SMD:C_0805_2012Metric, F.Cu at (123.6, 59.7)
- added C501: 1uF, Capacitor_SMD:C_0603_1608Metric, F.Cu at (67.8, 107.1)
- added C502: 1uF, Capacitor_SMD:C_0603_1608Metric, F.Cu at (67.8, 109.6)
- added C601: 2.2uF, Capacitor_SMD:C_0603_1608Metric, F.Cu at (218.1, 121.0)
- added C602: 100pf, Capacitor_SMD:C_0603_1608Metric, F.Cu at (218.1, 123.5)
- added C603: 2.2uF, Capacitor_SMD:C_0603_1608Metric, F.Cu at (218.1, 126.1)
- added C604: 4.7pf, Capacitor_SMD:C_0603_1608Metric, F.Cu at (218.1, 128.6)
- added C605: 100pf, Capacitor_SMD:C_0603_1608Metric, F.Cu at (194.6, 127.1)
- added C606: 47uF, Capacitor_SMD:C_1206_3216Metric, F.Cu at (212.7, 120.2)
- added C607: 47uF, Capacitor_SMD:C_1206_3216Metric, F.Cu at (213.2, 124.8)
- added C608: 47uF, Capacitor_SMD:C_1206_3216Metric, F.Cu at (213.2, 128.2)
- added C609: 47uF, Capacitor_SMD:C_1206_3216Metric, F.Cu at (213.2, 131.5)
- added C610: 2.2uF, Capacitor_SMD:C_0603_1608Metric, F.Cu at (81.1, 69.0)
- added C611: 100pf, Capacitor_SMD:C_0603_1608Metric, F.Cu at (81.1, 71.5)
- added C612: 2.2uF, Capacitor_SMD:C_0603_1608Metric, F.Cu at (85.1, 56.5)
- added C613: 4.7pf, Capacitor_SMD:C_0603_1608Metric, F.Cu at (85.1, 59.0)
- added C614: 100pf, Capacitor_SMD:C_0603_1608Metric, F.Cu at (85.1, 61.5)
- added C615: 47uF, Capacitor_SMD:C_1206_3216Metric, F.Cu at (76.2, 70.3)
- added C616: 47uF, Capacitor_SMD:C_1206_3216Metric, F.Cu at (76.2, 73.6)
- added C617: 47uF, Capacitor_SMD:C_1206_3216Metric, F.Cu at (76.2, 77.0)
- added C618: 47uF, Capacitor_SMD:C_1206_3216Metric, F.Cu at (76.2, 80.3)
- added C701: C_10nF, OEM:C_0603_1608Metric, F.Cu at (101.0, 28.7)
- added D1001: WHITE, LED_SMD:LED_0805_2012Metric, F.Cu at (46.2, 101.6)
- added D101: WHITE, LED_SMD:LED_0805_2012Metric, F.Cu at (53.4, 46.8)
- added D102: WHITE, LED_SMD:LED_0805_2012Metric, F.Cu at (53.4, 49.8)
- added D103: BLUE, LED_SMD:LED_0805_2012Metric, F.Cu at (53.4, 52.9)
- added D1101: LED_0805_Red, footprints:LED_0805_OEM, F.Cu at (85.1, 92.4)
- added D1102: LED_0805, footprints:LED_0805_OEM, F.Cu at (85.1, 95.2)
- added D1103: LED_0805_Amber, footprints:LED_0805_OEM, F.Cu at (85.1, 97.9)
- added D1104: LED_0805_Red, footprints:LED_0805_OEM, F.Cu at (85.1, 100.7)
- added D1105: LED_0805, footprints:LED_0805_OEM, F.Cu at (90.0, 92.4)
- added D1106: LED_0805_Red, footprints:LED_0805_OEM, F.Cu at (90.0, 95.2)
- added D1107: LED_0805_Amber, footprints:LED_0805_OEM, F.Cu at (90.0, 97.9)
- added D1108: LED_0805, footprints:LED_0805_OEM, F.Cu at (90.0, 100.7)
- added D1109: LED_0805_Red, footprints:LED_0805_OEM, F.Cu at (95.0, 92.4)
- added D1110: LED_0805, footprints:LED_0805_OEM, F.Cu at (95.0, 95.2)
- added D1111: LED_0805_Red, footprints:LED_0805_OEM, F.Cu at (95.0, 97.9)
- added D1112: LED_0805, footprints:LED_0805_OEM, F.Cu at (95.0, 100.7)
- added D1201: WHITE, LED_SMD:LED_0805_2012Metric, F.Cu at (31.4, 87.2)
- added D1301: WHITE, LED_SMD:LED_0805_2012Metric, F.Cu at (88.8, 123.8)
- added D1401: WHITE, LED_SMD:LED_0805_2012Metric, F.Cu at (46.2, 72.7)
- added D1501: WHITE, LED_SMD:LED_0805_2012Metric, F.Cu at (31.4, 72.7)
- added D1601: WHITE, LED_SMD:LED_0805_2012Metric, F.Cu at (31.4, 101.6)
- added D1701: WHITE, LED_SMD:LED_0805_2012Metric, F.Cu at (120.1, 32.3)
- added D1801: WHITE, LED_SMD:LED_0805_2012Metric, F.Cu at (119.9, 100.8)
- added D1901: WHITE, LED_SMD:LED_0805_2012Metric, F.Cu at (105.2, 46.7)
- added D2001: WHITE, LED_SMD:LED_0805_2012Metric, F.Cu at (46.2, 87.2)
- added D201: WHITE, LED_SMD:LED_0805_2012Metric, F.Cu at (31.4, 116.0)
- added D2101: WHITE, LED_SMD:LED_0805_2012Metric, F.Cu at (119.9, 115.2)
- added D2201: WHITE, LED_SMD:LED_0805_2012Metric, F.Cu at (120.1, 46.7)
- added D401: WHITE, LED_SMD:LED_0805_2012Metric, F.Cu at (118.7, 85.0)
- added D601: DZ2S082X0L, Diode_SMD:D_SOD-523, F.Cu at (75.2, 87.8)
- added D701: WHITE, LED_SMD:LED_0805_2012Metric, F.Cu at (105.2, 32.3)
- added F1001: 200mA_Fuse, Fuse:Fuse_1206_3216Metric, F.Cu at (46.8, 98.4)
- added F1201: 200mA_Fuse, Fuse:Fuse_1206_3216Metric, F.Cu at (32.0, 84.0)
- added F1301: 200mA_Fuse, Fuse:Fuse_1206_3216Metric, F.Cu at (89.4, 120.7)
- added F1401: 200mA_Fuse, Fuse:Fuse_1206_3216Metric, F.Cu at (46.8, 69.5)
- added F1501: 200mA_Fuse, Fuse:Fuse_1206_3216Metric, F.Cu at (32.0, 69.5)
- added F1601: 200mA_Fuse, Fuse:Fuse_1206_3216Metric, F.Cu at (32.0, 98.4)
- added F1701: 200mA_Fuse, Fuse:Fuse_1206_3216Metric, F.Cu at (120.6, 29.1)
- added F1801: 200mA_Fuse, Fuse:Fuse_1206_3216Metric, F.Cu at (120.5, 97.6)
- added F1901: 200mA_Fuse, Fuse:Fuse_1206_3216Metric, F.Cu at (105.8, 43.6)
- added F2001: 200mA_Fuse, Fuse:Fuse_1206_3216Metric, F.Cu at (46.8, 84.0)
- added F201: 200mA_Fuse, Fuse:Fuse_1206_3216Metric, F.Cu at (32.0, 112.9)
- added F2101: 200mA_Fuse, Fuse:Fuse_1206_3216Metric, F.Cu at (120.5, 112.1)
- added F2201: 200mA_Fuse, Fuse:Fuse_1206_3216Metric, F.Cu at (120.6, 43.6)
- added F701: 200mA_Fuse, Fuse:Fuse_1206_3216Metric, F.Cu at (105.8, 29.1)
- added J101: Conn_02x02_Counter_Clockwise, Connector_Molex:Molex_Micro-Fit_3.0_43045-0400_2x02_P3.00mm_Horizontal, F.Cu at (35.5, 47.2)
- added J102: Conn_01x02, Connector_Molex:Molex_Nano-Fit_105313-xx02_1x02_P2.50mm_Horizontal, F.Cu at (45.2, 40.0)
- added J103: Conn_02x05_Top_Bottom, Connector_Molex:Molex_Micro-Fit_3.0_43045-1000_2x05_P3.00mm_Horizontal, F.Cu at (29.7, 32.5)
- added J301: Conn_02x09_Counter_Clockwise, Connector_PinSocket_2.54mm:PinSocket_2x09_P2.54mm_Vertical, F.Cu at (224.6, 38.4)
- added J302: Conn_02x09_Counter_Clockwise, Connector_PinSocket_2.54mm:PinSocket_2x09_P2.54mm_Vertical, F.Cu at (324.6, 38.4)
- added J401: Conn_01x04_Socket, Connector_PinSocket_2.54mm:PinSocket_1x04_P2.54mm_Vertical, F.Cu at (119.1, 57.5)
- added J402: USB_C_Receptacle_USB2.0_16P, Connector_USB:USB_C_Receptacle_G-Switch_GT-USB-7051x, F.Cu at (98.6, 76.5)
- added J501: Conn_02x09_Counter_Clockwise, Connector_PinSocket_2.54mm:PinSocket_2x09_P2.54mm_Vertical, F.Cu at (274.6, 38.4)
- added JP1001: SolderJumper_2_Open, Jumper:SolderJumper-2_P1.3mm_Open_TrianglePad1.0x1.5mm, F.Cu at (50.6, 101.8)
- added JP1201: SolderJumper_2_Open, Jumper:SolderJumper-2_P1.3mm_Open_TrianglePad1.0x1.5mm, F.Cu at (35.8, 87.4)
- added JP1301: SolderJumper_2_Open, Jumper:SolderJumper-2_P1.3mm_Open_TrianglePad1.0x1.5mm, F.Cu at (93.2, 124.1)
- added JP1401: SolderJumper_2_Open, Jumper:SolderJumper-2_P1.3mm_Open_TrianglePad1.0x1.5mm, F.Cu at (50.6, 73.0)
- added JP1501: SolderJumper_2_Open, Jumper:SolderJumper-2_P1.3mm_Open_TrianglePad1.0x1.5mm, F.Cu at (35.8, 73.0)
- added JP1601: SolderJumper_2_Open, Jumper:SolderJumper-2_P1.3mm_Open_TrianglePad1.0x1.5mm, F.Cu at (35.8, 101.8)
- added JP1701: SolderJumper_2_Open, Jumper:SolderJumper-2_P1.3mm_Open_TrianglePad1.0x1.5mm, F.Cu at (124.4, 32.5)
- added JP1801: SolderJumper_2_Open, Jumper:SolderJumper-2_P1.3mm_Open_TrianglePad1.0x1.5mm, F.Cu at (124.3, 101.1)
- added JP1901: SolderJumper_2_Open, Jumper:SolderJumper-2_P1.3mm_Open_TrianglePad1.0x1.5mm, F.Cu at (109.6, 47.0)
- added JP2001: SolderJumper_2_Open, Jumper:SolderJumper-2_P1.3mm_Open_TrianglePad1.0x1.5mm, F.Cu at (50.6, 87.4)
- added JP201: SolderJumper_2_Open, Jumper:SolderJumper-2_P1.3mm_Open_TrianglePad1.0x1.5mm, F.Cu at (35.8, 116.3)
- added JP2101: SolderJumper_2_Open, Jumper:SolderJumper-2_P1.3mm_Open_TrianglePad1.0x1.5mm, F.Cu at (124.3, 115.5)
- added JP2201: SolderJumper_2_Open, Jumper:SolderJumper-2_P1.3mm_Open_TrianglePad1.0x1.5mm, F.Cu at (124.4, 47.0)
- added JP701: SolderJumper_2_Open, Jumper:SolderJumper-2_P1.3mm_Open_TrianglePad1.0x1.5mm, F.Cu at (109.6, 32.5)
- added L601: 22uH, Inductor_SMD:L_12x12mm_H4.5mm, F.Cu at (203.0, 126.9)
- added L602: 22uH, Inductor_SMD:L_12x12mm_H4.5mm, F.Cu at (66.0, 76.6)
- added Q401: 2N7002E, Package_TO_SOT_SMD:SOT-23, F.Cu at (107.6, 85.6)
- added Q601: SQ2337ES, Package_TO_SOT_SMD:SOT-23, F.Cu at (75.9, 84.4)
- added R1001: 33, Resistor_SMD:R_2512_6332Metric, F.Cu at (44.3, 94.3)
- added R1002: 100, Resistor_SMD:R_0603_1608Metric, F.Cu at (42.0, 100.5)
- added R1003: 100, OEM:R_0603_1608Metric, F.Cu at (42.0, 103.0)
- added R101: 60, Resistor_SMD:R_0603_1608Metric, F.Cu at (45.1, 51.5)
- added R102: 400, Resistor_SMD:R_0603_1608Metric, F.Cu at (45.1, 54.0)
- added R103: 10k, Resistor_SMD:R_0603_1608Metric, F.Cu at (45.1, 56.6)
- added R104: 10k, Resistor_SMD:R_0603_1608Metric, F.Cu at (49.1, 46.5)
- added R105: 10k, Resistor_SMD:R_0603_1608Metric, F.Cu at (49.1, 49.0)
- added R106: 60, Resistor_SMD:R_0603_1608Metric, F.Cu at (49.1, 51.5)
- added R107: 330, OEM:R_0603_1608Metric, F.Cu at (49.1, 54.0)
- added R108: 5k, OEM:R_0603_1608Metric, F.Cu at (49.1, 56.6)
- added R1101: 300, OEM:R_0603_1608Metric, F.Cu at (84.6, 103.3)
- added R1102: 120, OEM:R_0603_1608Metric, F.Cu at (84.6, 105.8)
- added R1103: 220, OEM:R_0603_1608Metric, F.Cu at (84.6, 108.3)
- added R1104: 300, OEM:R_0603_1608Metric, F.Cu at (84.6, 110.8)
- added R1105: 120, OEM:R_0603_1608Metric, F.Cu at (88.6, 103.3)
- added R1106: 300, OEM:R_0603_1608Metric, F.Cu at (88.6, 105.8)
- added R1107: 220, OEM:R_0603_1608Metric, F.Cu at (88.6, 108.3)
- added R1108: 120, OEM:R_0603_1608Metric, F.Cu at (88.6, 110.8)
- added R1109: 300, OEM:R_0603_1608Metric, F.Cu at (92.6, 103.3)
- added R1110: 120, OEM:R_0603_1608Metric, F.Cu at (92.6, 105.8)
- added R1111: 300, OEM:R_0603_1608Metric, F.Cu at (92.6, 108.3)
- added R1112: 120, OEM:R_0603_1608Metric, F.Cu at (92.6, 110.8)
- added R1201: 33, Resistor_SMD:R_2512_6332Metric, F.Cu at (29.5, 79.9)
- added R1202: 100, Resistor_SMD:R_0603_1608Metric, F.Cu at (27.1, 86.1)
- added R1203: 100, OEM:R_0603_1608Metric, F.Cu at (27.1, 88.6)
- added R1301: 33, Resistor_SMD:R_2512_6332Metric, F.Cu at (86.9, 116.6)
- added R1302: 100, Resistor_SMD:R_0603_1608Metric, F.Cu at (84.6, 122.8)
- added R1303: 100, OEM:R_0603_1608Metric, F.Cu at (84.6, 125.3)
- added R1401: 33, Resistor_SMD:R_2512_6332Metric, F.Cu at (44.3, 65.4)
- added R1402: 100, Resistor_SMD:R_0603_1608Metric, F.Cu at (42.0, 71.7)
- added R1403: 100, OEM:R_0603_1608Metric, F.Cu at (42.0, 74.2)
- added R1501: 33, Resistor_SMD:R_2512_6332Metric, F.Cu at (29.5, 65.4)
- added R1502: 100, Resistor_SMD:R_0603_1608Metric, F.Cu at (27.1, 71.7)
- added R1503: 100, OEM:R_0603_1608Metric, F.Cu at (27.1, 74.2)
- added R1601: 33, Resistor_SMD:R_2512_6332Metric, F.Cu at (29.5, 94.3)
- added R1602: 100, Resistor_SMD:R_0603_1608Metric, F.Cu at (27.1, 100.5)
- added R1603: 100, OEM:R_0603_1608Metric, F.Cu at (27.1, 103.0)
- added R1701: 33, Resistor_SMD:R_2512_6332Metric, F.Cu at (118.2, 25.0)
- added R1702: 100, Resistor_SMD:R_0603_1608Metric, F.Cu at (115.8, 31.2)
- added R1703: 100, OEM:R_0603_1608Metric, F.Cu at (115.8, 33.7)
- added R1801: 33, Resistor_SMD:R_2512_6332Metric, F.Cu at (118.0, 93.5)
- added R1802: 100, Resistor_SMD:R_0603_1608Metric, F.Cu at (115.6, 99.7)
- added R1803: 100, OEM:R_0603_1608Metric, F.Cu at (115.6, 102.2)
- added R1901: 33, Resistor_SMD:R_2512_6332Metric, F.Cu at (103.3, 39.5)
- added R1902: 100, Resistor_SMD:R_0603_1608Metric, F.Cu at (101.0, 45.7)
- added R1903: 100, OEM:R_0603_1608Metric, F.Cu at (101.0, 48.2)
- added R2001: 33, Resistor_SMD:R_2512_6332Metric, F.Cu at (44.3, 79.9)
- added R2002: 100, Resistor_SMD:R_0603_1608Metric, F.Cu at (42.0, 86.1)
- added R2003: 100, OEM:R_0603_1608Metric, F.Cu at (42.0, 88.6)
- added R201: 33, Resistor_SMD:R_2512_6332Metric, F.Cu at (29.5, 108.8)
- added R202: 100, Resistor_SMD:R_0603_1608Metric, F.Cu at (27.1, 115.0)
- added R203: 100, OEM:R_0603_1608Metric, F.Cu at (27.1, 117.5)
- added R2101: 33, Resistor_SMD:R_2512_6332Metric, F.Cu at (118.0, 108.0)
- added R2102: 100, Resistor_SMD:R_0603_1608Metric, F.Cu at (115.6, 114.2)
- added R2103: 100, OEM:R_0603_1608Metric, F.Cu at (115.6, 116.7)
- added R2201: 33, Resistor_SMD:R_2512_6332Metric, F.Cu at (118.2, 39.5)
- added R2202: 100, Resistor_SMD:R_0603_1608Metric, F.Cu at (115.8, 45.7)
- added R2203: 100, OEM:R_0603_1608Metric, F.Cu at (115.8, 48.2)
- added R301: 100k, Resistor_SMD:R_0603_1608Metric, F.Cu at (78.9, 26.3)
- added R302: 100k, Resistor_SMD:R_0603_1608Metric, F.Cu at (78.9, 28.8)
- added R303: 100k, Resistor_SMD:R_0603_1608Metric, F.Cu at (78.9, 31.3)
- added R304: 100k, Resistor_SMD:R_0603_1608Metric, F.Cu at (78.9, 33.9)
- added R305: 100k, Resistor_SMD:R_0603_1608Metric, F.Cu at (78.9, 36.4)
- added R306: 100k, Resistor_SMD:R_0603_1608Metric, F.Cu at (78.9, 38.9)
- added R307: 100k, Resistor_SMD:R_0603_1608Metric, F.Cu at (83.0, 23.8)
- added R308: 100k, Resistor_SMD:R_0603_1608Metric, F.Cu at (83.0, 26.3)
- added R309: 100k, Resistor_SMD:R_0603_1608Metric, F.Cu at (83.0, 28.8)
- added R310: 100k, Resistor_SMD:R_0603_1608Metric, F.Cu at (83.0, 31.3)
- added R311: 100k, Resistor_SMD:R_0603_1608Metric, F.Cu at (83.0, 33.9)
- added R312: 100k, Resistor_SMD:R_0603_1608Metric, F.Cu at (83.0, 36.4)
- added R313: 100k, Resistor_SMD:R_0603_1608Metric, F.Cu at (83.0, 38.9)
- added R314: 100k, Resistor_SMD:R_0603_1608Metric, F.Cu at (87.0, 23.8)
- added R315: 100k, Resistor_SMD:R_0603_1608Metric, F.Cu at (87.0, 26.3)
- added R316: 100k, Resistor_SMD:R_0603_1608Metric, F.Cu at (87.0, 28.8)
- added R317: 100k, Resistor_SMD:R_0603_1608Metric, F.Cu at (87.0, 31.3)
- added R318: 100k, Resistor_SMD:R_0603_1608Metric, F.Cu at (87.0, 33.9)
- added R319: 100k, Resistor_SMD:R_0603_1608Metric, F.Cu at (87.0, 36.4)
- added R320: 100k, Resistor_SMD:R_0603_1608Metric, F.Cu at (87.0, 38.9)
- added R321: 100k, Resistor_SMD:R_0603_1608Metric, F.Cu at (91.0, 23.8)
- added R322: 100k, Resistor_SMD:R_0603_1608Metric, F.Cu at (91.0, 26.3)
- added R323: 100k, Resistor_SMD:R_0603_1608Metric, F.Cu at (91.0, 28.8)
- added R324: 100k, Resistor_SMD:R_0603_1608Metric, F.Cu at (91.0, 31.3)
- added R325: 100k, Resistor_SMD:R_0603_1608Metric, F.Cu at (91.0, 33.9)
- added R326: 100k, Resistor_SMD:R_0603_1608Metric, F.Cu at (91.0, 36.4)
- added R327: 100k, Resistor_SMD:R_0603_1608Metric, F.Cu at (91.0, 38.9)
- added R328: 100k, Resistor_SMD:R_0603_1608Metric, F.Cu at (95.0, 23.8)
- added R329: 100k, Resistor_SMD:R_0603_1608Metric, F.Cu at (95.0, 26.3)
- added R330: 100k, Resistor_SMD:R_0603_1608Metric, F.Cu at (95.0, 28.8)
- added R331: 3.3k, Resistor_SMD:R_0603_1608Metric, F.Cu at (95.0, 31.3)
- added R332: 3.3k, Resistor_SMD:R_0603_1608Metric, F.Cu at (95.0, 33.9)
- added R401: 120, OEM:R_0603_1608Metric, F.Cu at (99.1, 71.5)
- added R402: 120, OEM:R_0603_1608Metric, F.Cu at (103.1, 56.5)
- added R403: 10k, footprints:R_0805_OEM, F.Cu at (123.4, 62.7)
- added R404: 100, footprints:R_0805_OEM, F.Cu at (123.4, 65.5)
- added R405: 5.1k, OEM:R_0603_1608Metric, F.Cu at (103.1, 59.0)
- added R406: 5.1k, OEM:R_0603_1608Metric, F.Cu at (103.1, 61.5)
- added R407: 5.1k, OEM:R_0603_1608Metric, F.Cu at (103.1, 64.0)
- added R408: 400, Resistor_SMD:R_0603_1608Metric, F.Cu at (103.1, 66.5)
- added R501: 20k, OEM:R_0603_1608Metric, F.Cu at (67.8, 112.2)
- added R502: 100, OEM:R_0603_1608Metric, F.Cu at (67.8, 114.7)
- added R601: 10k, Resistor_SMD:R_0603_1608Metric, F.Cu at (85.1, 64.0)
- added R602: 25.5k, Resistor_SMD:R_0603_1608Metric, F.Cu at (222.1, 131.1)
- added R603: 1M, Resistor_SMD:R_0603_1608Metric, F.Cu at (85.1, 69.0)
- added R604: 10k, Resistor_SMD:R_0603_1608Metric, F.Cu at (85.1, 71.5)
- added R605: 1M, Resistor_SMD:R_0603_1608Metric, F.Cu at (226.1, 121.0)
- added R606: 191k, Resistor_SMD:R_0603_1608Metric, F.Cu at (226.1, 123.5)
- added R607: 25.5k, Resistor_SMD:R_0603_1608Metric, F.Cu at (89.1, 61.5)
- added R608: 1M, Resistor_SMD:R_0603_1608Metric, F.Cu at (89.1, 64.0)
- added R609: 324k, Resistor_SMD:R_0603_1608Metric, F.Cu at (89.1, 66.5)
- added R701: 33, Resistor_SMD:R_2512_6332Metric, F.Cu at (103.3, 25.0)
- added R702: 100, Resistor_SMD:R_0603_1608Metric, F.Cu at (101.0, 31.2)
- added R703: 100, OEM:R_0603_1608Metric, F.Cu at (101.0, 33.7)
- added REF**: TestPoint_Pad_D4.0mm, TestPoint:TestPoint_Pad_D4.0mm, F.Cu at (338.1, 68.4)
- added REF**: TestPoint_Pad_D4.0mm, TestPoint:TestPoint_Pad_D4.0mm, F.Cu at (239.5, 36.4)
- added REF**: TestPoint_Pad_D4.0mm, TestPoint:TestPoint_Pad_D4.0mm, F.Cu at (289.5, 36.4)
- added SW401: SW_SPDT, Button_Switch_SMD:SW_SPDT_Shouhan_MSK12C02, F.Cu at (98.1, 83.6)
- added SW402: SW_MEC_5G, Button_Switch_SMD:SW_MEC_5GSH9, F.Cu at (110.9, 63.5)
- added TH301: Thermistor, Resistor_SMD:R_0603_1608Metric, F.Cu at (95.0, 36.4)
- added TP101: TP_SMD, TestPoint:TestPoint_Keystone_5019_Miniature, F.Cu at (28.0, 39.2)
- added TP102: TestPoint, TestPoint:TestPoint_Pad_1.0x1.0mm, F.Cu at (32.4, 53.5)
- added TP103: TP_SMD, TestPoint:TestPoint_Keystone_5019_Miniature, F.Cu at (28.0, 43.2)
- added TP104: TestPoint, TestPoint:TestPoint_Pad_1.0x1.0mm, F.Cu at (32.4, 56.6)
- added TP105: TP_SMD, TestPoint:TestPoint_Keystone_5019_Miniature, F.Cu at (28.0, 47.1)
- added TP106: TestPoint, TestPoint:TestPoint_Pad_1.0x1.0mm, F.Cu at (35.5, 53.5)
- added TP107: TP_SMD, TestPoint:TestPoint_Keystone_5019_Miniature, F.Cu at (28.0, 51.1)
- added TP108: TestPoint, TestPoint:TestPoint_Pad_1.0x1.0mm, F.Cu at (35.5, 56.6)
- added TP109: TP_SMD, TestPoint:TestPoint_Keystone_5019_Miniature, F.Cu at (28.0, 55.0)
- added TP110: TestPoint, TestPoint:TestPoint_Pad_1.0x1.0mm, F.Cu at (38.5, 53.5)
- added TP111: TP_SMD, TestPoint:TestPoint_Keystone_5019_Miniature, F.Cu at (28.0, 59.0)
- added TP112: TestPoint, TestPoint:TestPoint_Pad_1.0x1.0mm, F.Cu at (38.5, 56.6)
- added TP801: TestPoint, TestPoint:TestPoint_Pad_1.0x1.0mm, F.Cu at (41.5, 107.8)
- added TP802: TestPoint, TestPoint:TestPoint_Pad_1.0x1.0mm, F.Cu at (41.5, 110.9)
- added TP803: TestPoint, TestPoint:TestPoint_Pad_1.0x1.0mm, F.Cu at (41.5, 113.9)
- added TP804: TestPoint, TestPoint:TestPoint_Pad_1.0x1.0mm, F.Cu at (44.5, 107.8)
- added TP805: TestPoint, TestPoint:TestPoint_Pad_1.0x1.0mm, F.Cu at (44.5, 110.9)
- added TP806: TestPoint, TestPoint:TestPoint_Pad_1.0x1.0mm, F.Cu at (44.5, 113.9)
- added TP807: TestPoint, TestPoint:TestPoint_Pad_1.0x1.0mm, F.Cu at (47.6, 107.8)
- added TP808: TestPoint, TestPoint:TestPoint_Pad_1.0x1.0mm, F.Cu at (47.6, 110.9)
- added TP809: TestPoint, TestPoint:TestPoint_Pad_1.0x1.0mm, F.Cu at (47.6, 113.9)
- added TP810: TestPoint, TestPoint:TestPoint_Pad_1.0x1.0mm, F.Cu at (50.6, 107.8)
- added TP811: TestPoint, TestPoint:TestPoint_Pad_1.0x1.0mm, F.Cu at (50.6, 110.9)
- added TP812: TestPoint, TestPoint:TestPoint_Pad_1.0x1.0mm, F.Cu at (50.6, 113.9)
- added TP813: TestPoint, TestPoint:TestPoint_Pad_1.0x1.0mm, F.Cu at (53.7, 107.8)
- added TP814: TestPoint, TestPoint:TestPoint_Pad_1.0x1.0mm, F.Cu at (53.7, 110.9)
- added TP815: TestPoint, TestPoint:TestPoint_Pad_1.0x1.0mm, F.Cu at (53.7, 113.9)
- added TP901: TestPoint, TestPoint:TestPoint_Pad_1.0x1.0mm, F.Cu at (101.0, 92.6)
- added TP902: TestPoint, TestPoint:TestPoint_Pad_1.0x1.0mm, F.Cu at (101.0, 95.6)
- added TP903: TestPoint, TestPoint:TestPoint_Pad_1.0x1.0mm, F.Cu at (101.0, 98.7)
- added TP904: TestPoint, TestPoint:TestPoint_Pad_1.0x1.0mm, F.Cu at (101.0, 101.7)
- added TP905: TestPoint, TestPoint:TestPoint_Pad_1.0x1.0mm, F.Cu at (101.0, 104.8)
- added TP906: TestPoint, TestPoint:TestPoint_Pad_1.0x1.0mm, F.Cu at (101.0, 107.8)
- added TP907: TestPoint, TestPoint:TestPoint_Pad_1.0x1.0mm, F.Cu at (101.0, 110.9)
- added TP908: TestPoint, TestPoint:TestPoint_Pad_1.0x1.0mm, F.Cu at (104.0, 92.6)
- added TP909: TestPoint, TestPoint:TestPoint_Pad_1.0x1.0mm, F.Cu at (104.0, 95.6)
- added TP910: TestPoint, TestPoint:TestPoint_Pad_1.0x1.0mm, F.Cu at (104.0, 98.7)
- added TP911: TestPoint, TestPoint:TestPoint_Pad_1.0x1.0mm, F.Cu at (104.0, 101.7)
- added TP912: TestPoint, TestPoint:TestPoint_Pad_1.0x1.0mm, F.Cu at (104.0, 104.8)
- added TP913: TestPoint, TestPoint:TestPoint_Pad_1.0x1.0mm, F.Cu at (104.0, 107.8)
- added TP914: TestPoint, TestPoint:TestPoint_Pad_1.0x1.0mm, F.Cu at (104.0, 110.9)
- added TP915: TestPoint, TestPoint:TestPoint_Pad_1.0x1.0mm, F.Cu at (107.1, 92.6)
- added TP916: TestPoint, TestPoint:TestPoint_Pad_1.0x1.0mm, F.Cu at (107.1, 95.6)
- added TP917: TestPoint, TestPoint:TestPoint_Pad_1.0x1.0mm, F.Cu at (107.1, 98.7)
- added TP918: TestPoint, TestPoint:TestPoint_Pad_1.0x1.0mm, F.Cu at (107.1, 101.7)
- added TP919: TestPoint, TestPoint:TestPoint_Pad_1.0x1.0mm, F.Cu at (107.1, 104.8)
- added TP920: TestPoint, TestPoint:TestPoint_Pad_1.0x1.0mm, F.Cu at (107.1, 107.8)
- added TP921: TestPoint, TestPoint:TestPoint_Pad_1.0x1.0mm, F.Cu at (107.1, 110.9)
- added TP922: TestPoint, TestPoint:TestPoint_Pad_1.0x1.0mm, F.Cu at (110.1, 92.6)
- added TP923: TestPoint, TestPoint:TestPoint_Pad_1.0x1.0mm, F.Cu at (110.1, 95.6)
- added TP924: TestPoint, TestPoint:TestPoint_Pad_1.0x1.0mm, F.Cu at (110.1, 98.7)
- added TP925: TestPoint, TestPoint:TestPoint_Pad_1.0x1.0mm, F.Cu at (110.1, 101.7)
- added TP926: TestPoint, TestPoint:TestPoint_Pad_1.0x1.0mm, F.Cu at (110.1, 104.8)
- added TP927: TestPoint, TestPoint:TestPoint_Pad_1.0x1.0mm, F.Cu at (110.1, 107.8)
- added TP928: TestPoint, TestPoint:TestPoint_Pad_1.0x1.0mm, F.Cu at (110.1, 110.9)
- added U101: TSC2011IST, BAD_LIB:SO_011IST_STM-M, F.Cu at (50.6, 30.5)
- added U102: 74AHC1G08, OEM:SOT-23-5, F.Cu at (53.5, 56.7)
- added U103: LTV-356T, Package_SO:SO-4_4.4x3.6mm_P2.54mm, F.Cu at (51.3, 25.3)
- added U301: MAX14661ETI+T, BAD_LIB:21-0139I_T2844-1_MXM, F.Cu at (76.1, 43.3)
- added U302: MAX14661ETI+T, BAD_LIB:21-0139I_T2844-1_MXM, F.Cu at (76.1, 49.8)
- added U401: STM32G473CCTx, Package_QFP:LQFP-48_7x7mm_P0.5mm, F.Cu at (110.8, 77.5)
- added U402: TCAN1042VDRQ1, BAD_LIB:D0008A_M, F.Cu at (121.1, 75.4)
- added U403: USBLC6-2SC6, Package_TO_SOT_SMD:SOT-23-6, F.Cu at (119.0, 81.3)
- added U501: ADBMS1818, footprints:LQFP-64-1EP_12x12_P0.5, F.Cu at (73.2, 98.5)
- added U601: ~, BAD_LIB:SOP65P640X120-17N, F.Cu at (202.8, 138.3)
- added U602: ~, BAD_LIB:SOP65P640X120-17N, F.Cu at (84.1, 85.0)
- added Y401: 48 MHZ, footprints:Crystal_SMD_FA238, F.Cu at (112.6, 85.3)
- added kibuzzard-68FE9694: G***, kibuzzard-68FE9694, F.Cu at (314.5, 41.4)
- added kibuzzard-68FE96E6: G***, kibuzzard-68FE96E6, F.Cu at (214.5, 41.4)
- added kibuzzard-68FE9708: G***, kibuzzard-68FE9708, F.Cu at (264.5, 41.4)
Routing:
- added copper zone on In2.Cu, net +3.3V
- added copper zone on In1.Cu, net GND
Other:
- board outline added: 179 x 70 mm
- copper layers 2 -> 4

Commit message: some pcb layout
Parts:
- moved F201 281.5 mm to (282.5, 241.2)
- moved R201 281.5 mm to (280.0, 237.1)
- moved C201 281.5 mm to (277.7, 240.8)
- moved D201 281.5 mm to (281.9, 244.4)
- moved JP201 281.5 mm to (286.3, 244.6)
- moved R202 281.5 mm to (277.7, 243.3)
- moved R203 281.5 mm to (277.7, 245.8)
- moved C1201 270.9 mm to (276.6, 189.3)
- moved D1201 270.9 mm to (280.9, 192.9)
- moved F1201 270.9 mm to (281.4, 189.7)
- moved JP1201 270.9 mm to (285.2, 193.1)
- moved R1202 270.9 mm to (276.6, 191.8)
- moved R1203 270.9 mm to (276.6, 194.3)
- moved R1201 270.9 mm to (279.0, 185.6)
- moved C1501 267.9 mm to (286.2, 137.5), turned to -90 degrees
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