File: Hardware/Core/flight-core/flight-core.kicad_sch (KiCad schematic)
At the start: 9 parts, among them J1 CONN_02x03_RA, J101 Conn_01x02, J106 Conn_01x02, J107 Conn_01x02, J2 CONN_02x03_RA, J3 CONN_02x03_RA, J4 CONN_02x03_RA

Commit message: added df17 part to library, added stm32 actual names of pins
Parts:
- added R2: R_100K, footprints:R_0805_OEM, symbol formula:R_100K
- added U2: DC DC CONVERTER 12V 240W, symbol formula:DC_DC_CONVERTER_12V_240W
Connections:
- net +BATT_IN: now also U2.1 (+IN)
- net GND: now also R2.2, U2.3 (-IN)
- net at J101.2 (Pin_2): now also R2.1
Other:
- added sheet Cube connector (untitled.kicad_sch)
- moved on the sheet: J101

Commit message: adding cube connector
Other:
- sheet Cube connector: file untitled.kicad_sch -> cubeconnect.kicad_sch
Changed lines of the file:
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@@
 			)
 		)
-		(property "Sheetfile" "untitled.kicad_sch"
+		(property "Sheetfile" "cubeconnect.kicad_sch"
 			(at 193.675 84.4046 0)
 			(effects
